File: meter-board/meter-board.kicad_sch (KiCad schematic)
At the start: 149 parts, among them J1 2-1445053-2, J2 3-794636-8, J3 2-1445053-4, Q1 PMN100EPAX, Q2 2N7002K-AU_R1_000A2, U1 AP66300QFVBW-13, U2 TS431BIYLT, U3 ACSC02-41SURKWA-F01, U4 ACSC02-41SURKWA-F01, U5 ACSC02-41SURKWA-F01, U6 157121S12700, U7 157121S12700, U8 157121S12700

Commit message: modify pwr line
Connections:
- net +5VD: now also D8.2 (A); no longer D8.2  (A)
- net GND: no longer J1.MP1 (MountPin)
- net at C1.2, D1.2 (A2), FL1.2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: now also J1.MP1 (MountPin)
Changed lines of the file:
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@@
 	)
 	(junction
+		(at 40.64 35.56)
+		(diameter 0)
+		(color 0 0 0 0)
+	)
+	(junction
 		(at 76.2 45.72)
 		(diameter 0)
@@
 	(wire
 		(pts
-			(xy 127 228.6) (xy 137.16 228.6)
+			(xy 40.64 35.56) (xy 40.64 45.72)
 		)
 		(stroke
@@
 	(wire
 		(pts
-			(xy 27.94 15.24) (xy 30.48 15.24)
+			(xy 127 228.6) (xy 137.16 228.6)
 		)
 		(stroke
@@
 	(wire
 		(pts
+			(xy 12.7 15.24) (xy 30.48 15.24)
+		)
+		(stroke
+			(width 0)
+			(type default)
+		)
+	)
+	(wire
+		(pts
 			(xy 203.2 81.28) (xy 223.52 81.28)
 		)
@@
 	(wire
 		(pts
+			(xy 40.64 45.72) (xy 12.7 45.72)
+		)
+		(stroke
+			(width 0)
+			(type default)
+		)
+	)
+	(wire
+		(pts
 			(xy 147.32 147.32) (xy 147.32 149.86)
 		)
@@
 	(wire
 		(pts
+			(xy 12.7 45.72) (xy 12.7 15.24)
+		)
+		(stroke
+			(width 0)
+			(type default)
+		)
+	)
+	(wire
+		(pts
 			(xy 114.3 198.12) (xy 114.3 200.66)
 		)
@@
 	)
 	(symbol
-		(lib_id "my_Power:GND")
-		(at 27.94 15.24 270)
-		(unit 1)
-		(exclude_from_sim no)
-		(in_bom yes)
-		(on_board yes)
-		(dnp no)
-		(fields_autoplaced yes)
-		(property "Reference" "#PWR0138"
-			(at 21.59 15.24 0)
-			(effects
-				(font
-					(size 1.27 1.27)
-				)
-				(hide yes)
-			)
-		)
-		(property "Value" "GND"
-			(at 24.13 15.2399 90)
-			(effects
-				(font
-					(size 1.27 1.27)
-				)
-				(justify right)
-			)
-		)
-		(property "Footprint" ""
-			(at 27.94 15.24 0)
-			(effects
-				(font
-					(size 1.27 1.27)
-				)
-				(hide yes)
-			)
-		)
-		(property "Datasheet" ""
-			(at 27.94 15.24 0)
-			(effects
-				(font
-					(size 1.27 1.27)
-				)
-				(hide yes)
-			)
-		)
-		(property "Description" "Power symbol creates a global label with name \"GND\" , ground"
-			(at 27.94 15.24 0)
-			(effects
-				(font
-					(size 1.27 1.27)
-				)
-				(hide yes)
-			)
-		)
-		(pin "1"
-		)
-		(instances
-			(project "meter-board"
-				(path "/968e8a7b-5ca9-4f06-9bb4-2536f4d1b0b4"
-					(reference "#PWR0138")
-					(unit 1)
-				)
-			)
-		)
-	)
-	(symbol
 		(lib_id "my_Resistor:R_0402_1005M")
 		(at 246.38 50.8 0)
@@
 		(pin "4"
 		)
-		(pin "2\n"
+		(pin "2"
 		)
 		(pin "1"

Commit message: modify net name
Connections:
- net W5_W1 renamed W4_W1
- net W5_W2 renamed W4_W2
- net W5_W3 renamed W4_W4
- net W5_W4 renamed W4_W3
Other:
- sheet 7seg-and-led-driver ports: added W4_W1, W4_W2, W4_W3, W4_W4; removed W5_W1, W5_W2, W5_W3, W5_W4
Changed lines of the file:
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@@
 		)
 	)
-	(label "W5_W4"
-		(at 71.12 205.74 0)
+	(label "W4_W4"
+		(at 91.44 205.74 0)
 		(effects
 			(font
@@
 		)
 	)
-	(label "W5_W1"
+	(label "W4_W1"
 		(at 391.16 83.82 180)
 		(effects
@@
 		)
 	)
-	(label "W5_W2"
+	(label "W4_W2"
 		(at 50.8 205.74 0)
 		(effects
@@
 		)
 	)
-	(label "W5_W3"
+	(label "W4_W3"
 		(at 391.16 78.74 180)
 		(effects
@@
 		)
 	)
-	(label "W5_W4"
+	(label "W4_W4"
 		(at 391.16 76.2 180)
 		(effects
@@
 		)
 	)
-	(label "W5_W3"
-		(at 91.44 205.74 0)
+	(label "W4_W3"
+		(at 71.12 205.74 0)
 		(effects
 			(font
@@
 		)
 	)
-	(label "W5_W2"
+	(label "W4_W2"
 		(at 391.16 81.28 180)
 		(effects
@@
 		)
 	)
-	(label "W5_W1"
+	(label "W4_W1"
 		(at 30.48 205.74 0)
 		(effects
@@
 			)
 		)
-		(pin "W5_W1" output
-			(at 381 83.82 0)
-			(effects
-				(font
-					(size 1.27 1.27)
-				)
-				(justify right)
-			)
-		)
 		(pin "~{CS}" input
 			(at 355.6 30.48 180)
@@
 			)
 		)
-		(pin "W5_W2" output
-			(at 381 81.28 0)
+		(pin "R1_R1" output
+			(at 381 73.66 0)
 			(effects
 				(font
@@
 			)
 		)
-		(pin "W5_W3" output
-			(at 381 78.74 0)
+		(pin "W4_W1" output
+			(at 381 83.82 0)
 			(effects
 				(font
@@
 			)
 		)
-		(pin "W5_W4" output
+		(pin "W4_W4" output
 			(at 381 76.2 0)
 			(effects
@@
 			)
 		)
-		(pin "R1_R1" output
-			(at 381 73.66 0)
+		(pin "W4_W2" output
+			(at 381 81.28 0)
+			(effects
+				(font
+					(size 1.27 1.27)
+				)
+				(justify right)
+			)
+		)
+		(pin "W4_W3" output
+			(at 381 78.74 0)
 			(effects
 				(font
